Commit message: modify cars models

File: robot_launch/my_xacro/myrobot.urdf (robot description, URDF)
Before this commit: robot robot1_xacro, 10 links, 9 joints
Links:
- added link lever; visual cylinder length=0.4 radius=0.02
- added link motor1; visual cylinder length=0.18 radius=0.014
- added link motor2; visual cylinder length=0.18 radius=0.014
- added link motor3; visual cylinder length=0.18 radius=0.014
- added link motor4; visual cylinder length=0.18 radius=0.014
- link base_link: geometry collision box size=.5 .4 .09; visual box size=.5 .4 .09
Joints:
- added joint lever_joint: type fixed, parent base_link, child lever, origin xyz=-0.23 0 0.08 rpy=0 0 0
- added joint motor1_joint: type fixed, parent base_link, child motor1, origin xyz=0.23 0.15 -0.02 rpy=0 0 0
- added joint motor2_joint: type fixed, parent base_link, child motor2, origin xyz=-0.23 0.15 -0.02 rpy=0 0 0
- added joint motor3_joint: type fixed, parent base_link, child motor3, origin xyz=0.23 -0.15 -0.02 rpy=0 0 0
- added joint motor4_joint: type fixed, parent base_link, child motor4, origin xyz=-0.23 -0.15 -0.02 rpy=0 0 0
- joint base_to_wheel1: origin xyz=0.25 0.25 -0.05 rpy=1.5707 0 0 -> xyz=0.23 0.25 -0.05 rpy=1.5707 0 0
- joint base_to_wheel2: origin xyz=-0.25 0.25 -0.05 rpy=1.5707 0 0 -> xyz=-0.23 0.25 -0.05 rpy=1.5707 0 0
- joint base_to_wheel3: origin xyz=0.25 -0.25 -0.05 rpy=1.5707 0 0 -> xyz=0.23 -0.25 -0.05 rpy=1.5707 0 0
- joint base_to_wheel4: origin xyz=-0.25 -0.25 -0.05 rpy=1.5707 0 0 -> xyz=-0.23 -0.25 -0.05 rpy=1.5707 0 0
- joint horizontal_imu_link_1_joint: origin xyz=0 -0.1 0.2 rpy=0 0 0 -> xyz=-0.1 0 0.2 rpy=0 0 0
